Commit message: Use continuous wheel joints in sim models

File: src/navegacion_gps/models/cuatri_real.urdf (robot description, URDF)
Before this commit: robot quad_ackermann_viewer_safe, 11 links, 10 joints
Joints:
- joint front_left_wheel_joint: limit lower=-1000 upper=1000 effort=200 velocity=100 -> effort=200 velocity=100; type revolute -> continuous
- joint front_right_wheel_joint: limit lower=-1000 upper=1000 effort=200 velocity=100 -> effort=200 velocity=100; type revolute -> continuous
- joint rear_left_wheel_joint: limit lower=-1000 upper=1000 effort=200 velocity=100 -> effort=200 velocity=100; type revolute -> continuous
- joint rear_right_wheel_joint: limit lower=-1000 upper=1000 effort=200 velocity=100 -> effort=200 velocity=100; type revolute -> continuous
